File: kicad_frontpanel/kicad_frontpanel.kicad_pcb (KiCad board)
At the start: 2 copper layers, 30 x 128.5 mm, 19 parts

Commit message: version bump
Other:
- board text added: "rev 1.0 l-i-l.de"
- board text removed: "rev 0.3 l-i-l.de"
Changed lines of the file:
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@@
       (drillshape 0)
       (scaleselection 1)
-      (outputdirectory "../out/dots_fp_0.1.1/")
+      (outputdirectory "../out/dots_fp_1.0")
     )
   )
@@
   (gr_line locked (start 24.245249 22.706889) (end 24.256279 22.703216)
     (stroke (width 0.1) (type solid)) (layer "User.8"))
-  (gr_text "rev 0.3\nl-i-l.de" (at 31.05 137.2) (layer "B.SilkS")
+  (gr_text "rev 1.0\nl-i-l.de" (at 31.05 137.2) (layer "B.SilkS")
     (effects (font (size 0.8 0.8) (thickness 0.1) bold) (justify left bottom mirror))
   )

Commit message: pcb silkscreen rev bump
Other:
- board text added: "rev 0.1.0 l-i-l.de"
- board text removed: "rev 1.0 l-i-l.de"
Changed lines of the file:
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@@
   (gr_line locked (start 24.245249 22.706889) (end 24.256279 22.703216)
     (stroke (width 0.1) (type solid)) (layer "User.8"))
-  (gr_text "rev 1.0\nl-i-l.de" (at 31.05 137.2) (layer "B.SilkS")
+  (gr_text "rev 0.1.0\nl-i-l.de" (at 31.05 137.2) (layer "B.SilkS")
     (effects (font (size 0.8 0.8) (thickness 0.1) bold) (justify left bottom mirror))
   )
