File: kicad_main/peripheral.kicad_sch (KiCad schematic)
At the start: 6 parts, among them SW1 RotaryEncoder_Switch

Commit message: add missing potentiometer bom value
Parts:
- RV4-MOD1: value R_Potentiometer_US -> R_Potentiometer_US_100K
Changed lines of the file:
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@@
       (effects (font (size 1.27 1.27)) (justify right))
     )
-    (property "Value" "R_Potentiometer_US" (at 90.805 89.535 90)
+    (property "Value" "R_Potentiometer_US_100K" (at 90.805 89.535 90)
       (effects (font (size 1.27 1.27)) hide)
     )
